Commit message: update

File: kinova_description/urdf/j2s6s300.xacro (robot description, xacro)
@@ -65,5 +65,5 @@
     <xacro:property name="joint_3_upper_limit" value="${341/180*J_PI}" />
     <xacro:property name="joint_4" value="joint_4" />
-    <xacro:property name="joint_4_type" value="continuous" />
+    <xacro:property name="joint_4_type" value="continuous" />prefix
     <xacro:property name="joint_4_axis_xyz" value="0 0 1" />
     <xacro:property name="joint_4_origin_xyz" value="0 0.2073 -0.0114" />
